File: CyJTAG.kicad_pcb (KiCad board)
At the start: 2 copper layers, 33.7 x 21.6 mm, 8 parts, among them P1 USB_B, P2 CONN_01X10, P3 CONN_01X06, P4 CONN_01X06, U1 CY7C65215

Commit message: Updated schematic and layout
1. Added missing reset pull-up in layout
2. Made USB port mounting holes circular (for OSHPark)
3. Removed the default GPIO functions from the IC symbol
4. General layout cleanup
Parts:
- added R1: 4.7k, Resistors_SMD:R_0402, F.Cu at (116.8, 110.5)
Routing:
- net GND: track 64.3 -> 64.8 mm
- net VDD: track 41.1 -> 41.6 mm
